File: MomeaProbe12/Amplificador.kicad_sch (KiCad schematic)
At the start: 126 parts, among them J1 51K201-400N5, J2 51K201-400N5, U1 AD8065, U2 AD8065, U3 OPA847xDBV, U4 OPA847xDBV, U5 74HC4051, U6 74HC4051

Commit message: Adicionado informações sobre as etapas eletrônicas
Parts:
- C10, C22, C23, C41, C44, C8: value 2pF -> Placeholder
- C24, C25: value 10pF -> Placeholder
- C47, C54: value 6,8pF -> Placeholder
- L1, L2, L3, L4, L5, L6: value 10nH -> Placeholder
- R2, R4, R5, R6: value 50 -> Placeholder
- R29: value 120 -> 0
- R36: value 0 -> Placeholder
Other:
- moved on the sheet: C47, C48, C49, C50, C51, C52, C53, C54, C55, C56, C57, C58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
