File: MomeaProbe12/Fonte.kicad_sch (KiCad schematic)
At the start: 96 parts, among them J3-+5V-S1 +5V-S, J3-A3V3 A3V3, J3-GNDA1 GNDA, J4--5V-S1 -5V-S, J4-D3V3 3V3, J4-GNDREF1 GNDREF, U18 AD8065, U19 AD8065, U20 LM1117-3.3, U21 AD8065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

Commit message: Adicionado informações sobre as etapas eletrônicas
Other:
- moved on the sheet: C196, C197, C198, C199, C200, C201, C202, C203, C204, C205, C206, C207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
